File: proto-panel.kicad_pcb (KiCad board)
At the start: 4 copper layers, 180 x 125 mm, 1218 parts, among them J1 Conn_01x02_Socket, J2 Conn_01x02_Socket

Commit message: Final updates
Parts:
- removed the D194 at (223.6, 68.6)
- removed J1, J2: Conn_01x02_Socket, Connector_AMASS:AMASS_XT30U-F_1x02_P5.0mm_Vertical
- removed TP1, TP3, TP4, TP5, TP6, TP7, TP8: DO, TestPoint:TestPoint_Pad_D2.0mm
- added D732: LED, Custom Footprints:LED_WS2812B-2020_PLCC4_2.0x2.0mm-VIAPADS, F.Cu at (206.1, 110.6)
- added H10: MountingHole_Pad, MountingHole:MountingHole_2.2mm_M2_Pad, F.Cu at (210.6, 107.7)
- added H11: MountingHole_Pad, MountingHole:MountingHole_2.2mm_M2_Pad, F.Cu at (207.6, 115.1)
- added J3: Conn_01x08_Socket, Connector_FFC-FPC:Hirose_FH12-8S-0.5SH_1x08-1MP_P0.50mm_Horizontal, F.Cu at (57.9, 123.0)
- renumbered D195 to D194, D196 to D195, D197 to D196, D198 to D197, D199 to D198, D200 to D199, D201 to D200, D202 to D201, D203 to D202, D204 to D203, D205 to D204, D206 to D205, D207 to D206, D208 to D207, D209 to D208, D210 to D209, D211 to D210, D212 to D211, D213 to D212, D214 to D213, D215 to D214, D216 to D215, D217 to D216, D218 to D217, D219 to D218, D220 to D219, D221 to D220, D222 to D221, D223 to D222, D224 to D223, D225 to D224, D226 to D225, D227 to D226, D228 to D227, D229 to D228, D230 to D229, D231 to D230, D232 to D231, D233 to D232, D234 to D233, D235 to D234, D236 to D235, D237 to D236, D238 to D237, D239 to D238, D240 to D239, D241 to D240, D242 to D241, D243 to D242, D244 to D243, D245 to D244, D246 to D245, D247 to D246, D248 to D247, D249 to D248, D250 to D249, D251 to D250, D252 to D251, D253 to D252, D254 to D253, D255 to D254, D256 to D255, D257 to D256, D258 to D257, D259 to D258, D260 to D259, D261 to D260, D262 to D261, D263 to D262, D264 to D263, D265 to D264, D266 to D265, D267 to D266, D268 to D267, D269 to D268, D270 to D269, D271 to D270, D272 to D271, D273 to D272, D274 to D273, D275 to D274, D276 to D275, D277 to D276, D278 to D277, D279 to D278, D280 to D279, D281 to D280, D282 to D281, D283 to D282, D284 to D283, D285 to D284, D286 to D285, D287 to D286, D288 to D287, D289 to D288, D290 to D289, D291 to D290, D292 to D291, D293 to D292, D294 to D293, D295 to D294, D296 to D295, D297 to D296, D298 to D297, D299 to D298, D300 to D299, D301 to D300, D302 to D301, D303 to D302, D304 to D303, D305 to D304, D306 to D305, D307 to D306, D308 to D307, D309 to D308, D310 to D309, D311 to D310, D312 to D311, D313 to D312, D314 to D313, D315 to D314, D316 to D315, D317 to D316, D318 to D317, D319 to D318, D320 to D319, D321 to D320, D322 to D321, D323 to D322, D324 to D323, D325 to D324, D326 to D325, D327 to D326, D328 to D327, D329 to D328, D330 to D329, D331 to D330, D332 to D331, D333 to D332, D334 to D333, D335 to D334, D336 to D335, D337 to D336, D338 to D337, D339 to D338, D340 to D339, D341 to D340, D342 to D341, D343 to D342, D344 to D343, D345 to D344, D346 to D345, D347 to D346, D348 to D347, D349 to D348, D350 to D349, D351 to D350, D352 to D351, D353 to D352, D354 to D353, D355 to D354, D356 to D355, D357 to D356, D358 to D357, D359 to D358, D360 to D359, D361 to D360, D362 to D361, D363 to D362, D364 to D363, D365 to D364, D366 to D365, D367 to D366, D368 to D367, D369 to D368, D370 to D369, D371 to D370, D372 to D371, D373 to D372, D374 to D373, D375 to D374, D376 to D375, D377 to D376, D378 to D377, D379 to D378, D380 to D379, D381 to D380, D382 to D381, D383 to D382, D384 to D383, D385 to D384, D386 to D385, D387 to D386, D388 to D387, D389 to D388, D390 to D389, D391 to D390, D392 to D391, D393 to D392, D394 to D393, D395 to D394, D396 to D395, D397 to D396, D398 to D397, D399 to D398, D400 to D399, D401 to D400, D402 to D401, D403 to D402, D404 to D403, D405 to D404, D406 to D405, D407 to D406, D408 to D407, D409 to D408, D410 to D409, D411 to D410, D412 to D411, D413 to D412, D414 to D413, D415 to D414, D416 to D415, D417 to D416, D418 to D417, D419 to D418, D420 to D419, D421 to D420, D422 to D421, D423 to D422, D424 to D423, D425 to D424, D426 to D425, D427 to D426, D428 to D427, D429 to D428, D430 to D429, D431 to D430, D432 to D431, D433 to D432, D434 to D433, D435 to D434, D436 to D435, D437 to D436, D438 to D437, D439 to D438, D440 to D439, D441 to D440, D442 to D441, D443 to D442, D444 to D443, D445 to D444, D446 to D445, D447 to D446, D448 to D447, D449 to D448, D450 to D449, D451 to D450, D452 to D451, D453 to D452, D454 to D453, D455 to D454, D456 to D455, D457 to D456, D458 to D457, D459 to D458, D460 to D459, D461 to D460, D462 to D461, D463 to D462, D464 to D463, D465 to D464, D466 to D465, D467 to D466, D468 to D467, D469 to D468, D470 to D469, D471 to D470, D472 to D471, D473 to D472, D474 to D473, D475 to D474, D476 to D475, D477 to D476, D478 to D477, D479 to D478, D480 to D479, D481 to D480, D482 to D481, D483 to D482, D484 to D483, D485 to D484, D486 to D485, D487 to D486, D488 to D487, D489 to D488, D490 to D489, D491 to D490, D492 to D491, D493 to D492, D494 to D493, D495 to D494, D496 to D495, D497 to D496, D498 to D497, D499 to D498, D500 to D499, D501 to D500, D502 to D501, D503 to D502, D504 to D503, D505 to D504, D506 to D505, D507 to D506, D508 to D507, D509 to D508, D510 to D509, D511 to D510, D512 to D511, D513 to D512, D514 to D513, D515 to D514, D516 to D515, D517 to D516, D518 to D517, D519 to D518, D520 to D519, D521 to D520, D522 to D521, D523 to D522, D524 to D523, D525 to D524, D526 to D525, D527 to D526, D528 to D527, D529 to D528, D530 to D529, D531 to D530, D532 to D531, D533 to D532, D534 to D533, D535 to D534, D536 to D535, D537 to D536, D538 to D537, D539 to D538, D540 to D539, D541 to D540, D542 to D541, D543 to D542, D544 to D543, D545 to D544, D546 to D545, D547 to D546, D548 to D547, D549 to D548, D550 to D549, D551 to D550, D552 to D551, D553 to D552, D554 to D553, D555 to D554, D556 to D555, D557 to D556, D558 to D557, D559 to D558, D560 to D559, D561 to D560, D562 to D561, D563 to D562, D564 to D563, D565 to D564, D566 to D565, D567 to D566, D568 to D567, D569 to D568, D570 to D569, D571 to D570, D572 to D571, D573 to D572, D574 to D573, D575 to D574, D576 to D575, D577 to D576, D578 to D577, D579 to D578, D580 to D579, D581 to D580, D582 to D581, D583 to D582, D584 to D583, D585 to D584, D586 to D585, D587 to D586, D588 to D587, D589 to D588, D590 to D589, D591 to D590, D592 to D591, D593 to D592, D594 to D593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
Connections:
- D194 pad 3: Net-(D194-DOUT) (its old number) -> Net-(D193-DOUT)
- D299 pad 1: unconnected-(D300-DOUT-Pad1) -> Net-(D299-DOUT)
- D300 pad 1: Net-(D301-DOUT) (its old number) -> unconnected-(D300-DOUT-Pad1)
- D300 pad 3: STR3 -> Net-(D299-DOUT)
- D301 pad 3: Net-(D301-DOUT) (its old number) -> STR3
- D449 pad 1: unconnected-(D450-DOUT-Pad1) -> Net-(D449-DOUT)
- D450 pad 1: Net-(D451-DOUT) (its old number) -> unconnected-(D450-DOUT-Pad1)
- D450 pad 3: STR4 -> Net-(D449-DOUT)
- D451 pad 3: Net-(D451-DOUT) (its old number) -> STR4
- D599 pad 1: unconnected-(D600-DOUT-Pad1) -> Net-(D599-DOUT)
- D600 pad 1: Net-(D601-DOUT) (its old number) -> unconnected-(D600-DOUT-Pad1)
- D600 pad 3: STR5 -> Net-(D599-DOUT)
- D601 pad 3: Net-(D601-DOUT) (its old number) -> STR5
- D731 pad 1: Net-(D732-DOUT) -> Net-(D731-DOUT)
Routing:
- net STR4: track 0.00 -> 151.7 mm, vias 0 -> 2
- net STR7: track 0.00 -> 149.0 mm, vias 0 -> 2
- net Net-(D194-DOUT) (its old number): track 135.8 -> 0.00 mm
- net Net-(D193-DOUT): track 2.13 -> 132.3 mm
- net STR3: track 0.00 -> 125.1 mm, vias 1 -> 2
- net STR2: track 43.9 -> 159.9 mm, vias 1 -> 2
- net STR8: track 0.00 -> 108.7 mm, vias 0 -> 2
- net STR1: track 71.8 -> 165.9 mm, vias 1 -> 2
- net STR6: track 0.00 -> 67.1 mm, vias 0 -> 2
- net Net-(D37-DOUT): track 0.00 -> 62.3 mm
- net STR5: track 0.00 -> 25.3 mm, vias 0 -> 2
- net unconnected-(D1200-DOUT-Pad1): track 14.3 -> 0.00 mm, vias 1 -> 0
- net Net-(D732-DOUT): track 153.3 -> 156.8 mm
- net Net-(D299-DOUT): track 0.00 -> 2.13 mm
- net Net-(D451-DOUT) (its old number): track 2.13 -> 0.00 mm
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Other:
- board text added: "+5V"
- board text added: "GND"
