File: proto-panel.kicad_sch (KiCad schematic)
At the start: 1219 parts, among them J1 Conn_01x02_Socket, J2 Conn_01x02_Socket

Commit message: Final updates
Parts:
- removed J1, J2: Conn_01x02_Socket, Connector_AMASS:AMASS_XT30U-F_1x02_P5.0mm_Vertical, symbol Connector:Conn_01x02_Socket
- removed TP1, TP2, TP3, TP4, TP5, TP6, TP7, TP8: DO, TestPoint:TestPoint_Pad_D2.0mm, symbol Connector:TestPoint
- added H10, H11: MountingHole_Pad, MountingHole:MountingHole_2.2mm_M2_Pad, symbol Mechanical:MountingHole_Pad
- added J3: Conn_01x08_Socket, Connector_FFC-FPC:Hirose_FH12-8S-0.5SH_1x08-1MP_P0.50mm_Horizontal, symbol Connector:Conn_01x08_Socket
Connections:
- net +5V: now also H10.1
- net GND: now also H11.1
- net STR1: now also J3.1 (Pin_1)
- net STR2: now also J3.2 (Pin_2)
- net STR3: now also J3.3 (Pin_3)
- net STR4: now also J3.4 (Pin_4)
- net STR5: now also J3.5 (Pin_5)
- net STR6: now also J3.6 (Pin_6)
- net STR7: now also J3.7 (Pin_7)
- net STR8: now also J3.8 (Pin_8)
